Commit message: Refine Astro hand, foot and neck-handle collision geometry

File: robots/astro_p2_29dof/astro_p2_29dof.urdf (robot description, URDF)
Before this commit: robot astro_p2_29dof, 37 links, 36 joints
Links:
- added link left_foot_link; collision box size=0.106 0.076 0.028; collision cylinder length=0.028 radius=0.041
- added link right_foot_link; collision box size=0.106 0.076 0.028; collision cylinder length=0.028 radius=0.041
- link left_ankle_roll_link: geometry visual mesh filename=meshes/left_ankle_roll_link.stl
- link left_hand_link: geometry collision sphere radius=0.027; visual sphere radius=0.027
- link left_wrist_yaw_link: geometry collision cylinder length=0.03 radius=0.027; visual mesh filename=meshes/left_wrist_yaw_link.stl
- link right_ankle_roll_link: geometry visual mesh filename=meshes/right_ankle_roll_link.stl
- link right_hand_link: geometry collision sphere radius=0.027; visual sphere radius=0.027
- link right_wrist_yaw_link: geometry collision cylinder length=0.03 radius=0.027; visual mesh filename=meshes/right_wrist_yaw_link.stl
- link waist_roll_link: geometry collision cylinder length=0.02 radius=0.09; collision cylinder length=0.04 radius=0.0075
Joints:
- added joint left_foot_joint: type fixed, parent left_ankle_roll_link, child left_foot_link, origin xyz=0 0 0 rpy=0 0 0
- added joint right_foot_joint: type fixed, parent right_ankle_roll_link, child right_foot_link, origin xyz=0 0 0 rpy=0 0 0

Commit message: Add native-capsule Astro MJCF and refine neck-handle supports

File: robots/astro_p2_29dof/astro_p2_29dof.urdf (robot description, URDF)
Before this commit: robot astro_p2_29dof, 39 links, 38 joints
Links:
- link waist_roll_link: geometry collision cylinder length=0.02 radius=0.09; collision cylinder length=0.035 radius=0.0075
